File: dataflyer-2650.kicad_sch (KiCad schematic)
At the start: 2 parts, among them J1 26-pin IDC (Dataflyer side), J2 50-pin IDC (SCSI chain out)

Commit message: 1.1.1: project text variables + silkscreen overhaul + J1 pin 1 marker
Project text variables (.kicad_pro):
- BOARD_NAME = "DataFlyer 2650 — 26-pin to 50-pin SCSI Adapter"
- BOARD_REV  = "1.1.1"
- sch_revision now references ${BOARD_REV}
- Plot output directory set to gerbers/

Schematic (.kicad_sch):
- title and rev fields now reference ${BOARD_NAME} / ${BOARD_REV}
  so the project text variables are the single source of truth

PCB (.kicad_pcb):
- Board-level BOARD_NAME and BOARD_REV properties added
- Front silkscreen overhauled:
  * Board name now uses ${BOARD_NAME} (fixes lingering lowercase
    "Dataflyer 2650 SCSI Adapter" instance)
  * Added "Rev ${BOARD_REV}" line
  * Added "github.com/arnljot/dataflyer2650" repo URL
  * Attribution split into two readable lines:
    "based on work by highpuff @ ikod.se" / "ikod.se/scsi-cable"
- J1 pin 1 marker added on B.Cu (bottom copper, mirrored, bold 1.5mm)
  for permanent indication on the underside that mates with the
  controller card's male header
- Plot output directory set to gerbers/

Patch release per the new release policy: lives on main, no GitHub
release tag.

(c) 2026 Arnljot Arntsen
Other:
- title: DataFlyer 2650 — 26-pin to 50-pin SCSI Adapter -> ${BOARD_NAME}
Changed lines of the file:
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@@
 	(paper "A5")
 	(title_block
-		(title "DataFlyer 2650 — 26-pin to 50-pin SCSI Adapter")
+		(title "${BOARD_NAME}")
 		(date "2026-06-02")
-		(rev "1.1")
+		(rev "${BOARD_REV}")
 		(comment 1 "For DataFlyer 1200 SCSI+ And Phase5 Blizzard IV SCSI kit")
 		(comment 2 "Based on SCSI cable by highpuff iKod.se")
